File: VCOMLCD.sch (KiCad schematic (older format))
At the start: 49 parts, among them J1 Screw_Terminal_01x02, J2 USB_B_Mini, J3 Conn_01x05, J4 Conn_01x03, J5 Conn_01x06, Q1 BC847, SW1 SYS_RST, SW2 BTN, U1 MCP73831-2-OT, U2 MCP1700-3302E_SOT23, U3 74LVC4245A, U4 LCD-016N002L, U5 STM32F042F4Px, U6 ESP-12E

Commit message: pre-fabrication commit
Parts:
- removed J1: Screw_Terminal_01x02, TerminalBlock_4Ucon:TerminalBlock_4Ucon_1x02_P3.50mm_Horizontal, symbol Connector:Screw_Terminal_01x02
- removed J3: Conn_01x05, Connector_PinHeader_2.54mm:PinHeader_1x05_P2.54mm_Horizontal, symbol Connector_Generic:Conn_01x05
- removed J4: Conn_01x03, Connector_PinHeader_2.54mm:PinHeader_1x03_P2.54mm_Horizontal, symbol Connector_Generic:Conn_01x03
- removed J5: Conn_01x06, Connector_PinHeader_2.54mm:PinHeader_1x06_P2.54mm_Horizontal, symbol Connector_Generic:Conn_01x06
- removed Q1: BC847, Package_TO_SOT_SMD:SOT-23, symbol Transistor_BJT:BC847
- removed SW1: SYS_RST, Button_Switch_THT:SW_Tactile_SPST_Angled_PTS645Vx83-2LFS, symbol Switch:SW_Push
- removed U2: MCP1700-3302E_SOT23, Package_TO_SOT_SMD:SOT-23, symbol Regulator_Linear:MCP1700-3302E_SOT23
- removed U5: STM32F042F4Px, Package_SO:TSSOP-20_4.4x6.5mm_P0.65mm, symbol MCU_ST_STM32F0:STM32F042F4Px
- removed U6: ESP-12E, RF_Module:ESP-12E, symbol RF_Module:ESP-12E
- added C14: 10u, Capacitor_SMD:C_1206_3216Metric_Pad1.42x1.75mm_HandSolder, symbol Device:C_Small
- added D1: LED_RED, LED_SMD:LED_0805_2012Metric_Pad1.15x1.40mm_HandSolder, symbol Device:LED
- added D2: LED_GREEN, LED_SMD:LED_0805_2012Metric_Pad1.15x1.40mm_HandSolder, symbol Device:LED
- added D3: LED_BLUE, LED_SMD:LED_0805_2012Metric_Pad1.15x1.40mm_HandSolder, symbol Device:LED
- added J1, J3: Conn_01x08, Connector_PinSocket_2.54mm:PinSocket_1x08_P2.54mm_Vertical, symbol Connector_Generic:Conn_01x08
- added J4: LiPo_ext, Connector_PinHeader_2.54mm:PinHeader_2x02_P2.54mm_Vertical, symbol Connector_Generic:Conn_02x02_Odd_Even
- added J5: Screw_Terminal_01x02, TerminalBlock:TerminalBlock_bornier-2_P5.08mm, symbol Connector:Screw_Terminal_01x02
- added Q1: BC817, Package_TO_SOT_SMD:SOT-23, symbol Transistor_BJT:BC817
- added Q2: AO3401A, Package_TO_SOT_SMD:SOT-23, symbol Transistor_FET:AO3401A
- added Q3: FS8205A, Package_SO:TSSOP-8_4.4x3mm_P0.65mm, symbol LiPo_protection:FS8205A
- added R20, R31: 1k, Resistor_SMD:R_0603_1608Metric_Pad1.05x0.95mm_HandSolder, symbol Device:R
- added R21, R32: 200, Resistor_SMD:R_0603_1608Metric_Pad1.05x0.95mm_HandSolder, symbol Device:R
- added R22, R25, R29, R30, R33: NC, Resistor_SMD:R_0603_1608Metric_Pad1.05x0.95mm_HandSolder, symbol Device:R
- added R23: 698k, Resistor_SMD:R_0603_1608Metric_Pad1.05x0.95mm_HandSolder, symbol Device:R
- added R24: 133k, Resistor_SMD:R_0603_1608Metric_Pad1.05x0.95mm_HandSolder, symbol Device:R
- added R26, R27: 10k/1%, Resistor_SMD:R_0603_1608Metric_Pad1.05x0.95mm_HandSolder, symbol Device:R
- added R28: 10k, Resistor_SMD:R_0603_1608Metric_Pad1.05x0.95mm_HandSolder, symbol Device:R
- added TP1: Lipo+, TestPoint:TestPoint_Pad_1.0x1.0mm, symbol Connector:TestPoint
- added TP2: LiPo-, TestPoint:TestPoint_Pad_1.0x1.0mm, symbol Connector:TestPoint
- added U2: ESP32-WROOM-32, RF_Module:ESP32-WROOM-32, symbol RF_Module:ESP32-WROOM-32
- added U5: XC6220B331MR, Package_TO_SOT_SMD:SOT-23-5, symbol Regulator_Linear:XC6220B331MR
- added U6: TLV61046ADB, Package_TO_SOT_SMD:SOT-23-6, symbol Regulator_Switching:TLV61046ADB
- added U7: DW01x, Package_TO_SOT_SMD:SOT-23-6, symbol LiPo_protection:DW01x
- C10, C3: value 100n -> 1u
- C11, C13, C2: value 22u -> 10u
- C4: value 22u -> 100n; footprint Capacitor_SMD:C_1206_3216Metric_Pad1.42x1.75mm_HandSolder -> Capacitor_SMD:C_0603_1608Metric_Pad1.05x0.95mm_HandSolder
- L1: value L_Small -> 0R
- L2: value L_Small -> 10uH
- R1: value NC -> 0R
- R13: value R -> 1k
- R16, R3, R8: value R -> 10k
- R2: value 0R -> 200
- RV1: footprint Potentiometer_SMD:Potentiometer_Vishay_TS53YJ_Vertical -> Potentiometer_THT:Potentiometer_Runtron_RM-065_Vertical
- U3: symbol Logic_LevelTranslator:74LVC4245A -> VCOMLCD-rescue:74LVC4245A-Logic_LevelTranslator
- U4: footprint Display:LCD-016N002L -> Display:WC1602A
Connections:
- net +3V3: now also C2.1, D3.2 (A), J1.3 (Pin_3), J3.8 (Pin_8), U2.2 (VDD), U5.5 (VOUT); no longer C3.1, C4.1, C8.1, C9.1
- net +BATT: now also C10.1, L2.1, J4.1 (Pin_1), J4.3 (Pin_3), Q2.3 (D), R28.2, R32.2, TP1.1, U6.6 (VI)
- net BL_CTRL: now also U2.37 (IO23); no longer R17.2
- net BTN: now also U2.7 (IO35)
- net GND: now also J2.5 (GND), J2.6 (Shield), R13.2, C14.2, J1.2 (Pin_2), J1.8 (Pin_8), J3.1 (Pin_1), J5.2 (Pin_2), Q1.2 (E), Q3.2 (S1), Q3.3 (S1), R24.2, R27.1, R30.1, R31.2, R33.1, U2.1 (GND), U2.15 (GND), U2.38 (GND), U2.39 (GND), U5.2 (GND), U6.2 (GND); no longer C4.2, C9.2, L2.2, R13.1
- net VBUS: now also D1.2 (A), D2.2 (A), J1.1 (Pin_1), R22.2, R25.2; no longer C6.1, C7.1, R2.2, RV1.1, U3.1 (VCCA), U4.15 (A/VEE), U4.2 (VDD)
- net E_3V3: now reaches U3.18 (B3)
- net E_3V3: now also U2.29 (IO5)
- net DB4_3V3: now reaches U3.17 (B4)
- net DB4_3V3: now also U2.30 (IO18)
- net DB5_3V3: now reaches U3.16 (B5)
- net DB5_3V3: now also U2.31 (IO19)
- net at J2.3 (D+): now also R2.1
- net at J2.2 (D-): now also R2.2
- net at U3.21 (B0): now also R18.2
- net at U3.20 (B1): now also R19.2
- net RS_3V3: now reaches U3.19 (B2)
- net RS_3V3: now also U2.28 (IO17)
- net at J2.1 (VBUS), L1.2: now also J5.1 (Pin_1)
- net at U4.11 (DB4): now also U3.7 (A4); no longer U3.3 (A0)
- net at U4.12 (DB5): now also U3.8 (A5); no longer U3.4 (A1)
- net at U4.13 (DB6): now also U3.10 (A7); no longer U3.5 (A2)
- net at U4.14 (DB7): now also U3.9 (A6); no longer U3.6 (A3)
- net at U4.16 (K): now also Q1.3 (C)
- net at RV1.2, U4.3 (VO): now also R29.1, R30.2
- net at U4.4 (RS): now also U3.5 (A2); no longer U3.8 (A5)
- net at U4.6 (E): now also U3.6 (A3); no longer U3.7 (A4)
- net at R12.1: now also R17.2, Q1.1 (B)
- net at R14.1: now also U2.24 (IO2)
- net at U1.1 (STAT): now also R20.2
- net DB6_3V3: now reaches U3.14 (B7)
- net DB6_3V3: now also U2.36 (IO22); no longer R19.2
- net DB7_3V3: now reaches U3.15 (B6)
- net DB7_3V3: now also U2.33 (IO21); no longer R18.2
- net ESP_DTR renamed PROG_DTR
- net PROG_DTR: now also J1.5 (Pin_5), U2.25 (IO0)
- net ESP_RTS renamed PROG_RTS
- net PROG_RTS: now also C8.1, J1.4 (Pin_4), U2.3 (EN); no longer C10.1
- new net: C3.1, R1.1, R22.1, U5.1 (VIN), U5.3 (CE)
- new net: R21.1, U2.23 (IO15)
- new net: L2.2, U6.1 (SW)
- new net: R23.2, R24.1, U6.3 (FB)
- new net: Q3.1 (D12), Q3.8 (D12)
- new net: Q3.4 (G1), U7.3 (OC)
- new net: Q3.5 (G2), U7.1 (OD)
- new net: C4.2, J4.2 (Pin_2), J4.4 (Pin_4), Q3.6 (S2), Q3.7 (S2), R33.2, TP2.1, U7.6 (GND)
- new net: R31.1, U7.2 (CS)
- new net: C4.1, R32.1, U7.5 (VCC)
- new net: D3.1 (K), R21.2
- new net: D1.1 (K), R13.1
- new net: D2.1 (K), R20.1
- new net: C9.1, Q2.1 (G), R28.1
- new net: Q2.2 (S), R26.2
- new net +5V: C14.1, C6.1, C7.1, R23.1, R25.1, R29.2, RV1.1, U3.1 (VCCA), U4.15 (A/VEE), U4.2 (VDD), U6.5 (VOUT)
- new net 5V_ENA: U2.16 (IO13), U6.4 (EN)
- new net GPIO12: J3.2 (Pin_2), U2.14 (IO12)
- new net GPIO14: J3.3 (Pin_3), U2.13 (IO14)
- new net GPIO25: J3.6 (Pin_6), U2.10 (IO25)
- new net GPIO26: J3.5 (Pin_5), U2.11 (IO26)
- new net GPIO27: J3.4 (Pin_4), U2.12 (IO27)
- new net GPIO33: J3.7 (Pin_7), U2.9 (IO33)
- new net LIPO_DIV: R26.1, R27.2, U2.8 (IO32)
- new net LIPO_DIV_ENA: C9.2, U2.26 (IO4)
- new net PROG_RXD: J1.6 (Pin_6), U2.35 (TXD0/IO1)
- new net PROG_TXD: J1.7 (Pin_7), U2.34 (RXD0/IO3)
- no-connect marks 0 -> 18
Other:
- note added: "For non-battery devices, this\npart may be left unpopulated"
- note added: "Rev. 1\n-Initial release\nRev.2\n- Changed focus of the project to battery-\npowered, with external\nprogrammer\n- Selected proper LCD footprint\n- Changed MCU to ESP32\n- added dedicated 5V pin\n- addded pwr/chr/gpio LEDs\n"
- note removed: "Rev. 1\n-Initial release\nRev.2\n- Selected proper LCD footprint\n- added dedicated 5V pin\n- removed R1/R2 solderbridges\n- addded pwr/status LEDs\n"
- moved on the sheet: C1, C11, C12, C13, C2, C3, C5, C6, C7, J2, L1, R1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

Commit message: oh darn, how old is this repo
Parts:
- U3: symbol VCOMLCD-rescue:74LVC4245A-Logic_LevelTranslator -> VCOMLCD-rescue:74LVC4245A-Logic_LevelTranslator-VCOMLCD-rescue
Connections:
- net +3V3: now also J1.1 (Pin_1); no longer J1.3 (Pin_3)
- net GND: now also J1.6 (Pin_6), J1.7 (Pin_7); no longer J1.2 (Pin_2), J1.8 (Pin_8)
- net PROG_DTR: now also J1.3 (Pin_3); no longer J1.5 (Pin_5)
- net PROG_RTS: now also J1.2 (Pin_2); no longer J1.4 (Pin_4)
- net PROG_RXD: now also J1.4 (Pin_4); no longer J1.6 (Pin_6)
- net PROG_TXD: now also J1.5 (Pin_5); no longer J1.7 (Pin_7)
- net VBUS: now also J1.8 (Pin_8); no longer J1.1 (Pin_1)
Other:
- moved on the sheet: J1
Changed lines of the file:
@@
 $EndComp
 Wire Wire Line
-	3950 3700 3850 3700
+	3950 3350 3850 3350
 $Comp
 L power:GND #PWR053
 U 1 1 5CEB4B4B
-P 3850 3900
-F 0 "#PWR053" H 3850 3650 50  0001 C CNN
-F 1 "GND" H 3855 3727 50  0000 C CNN
-F 2 "" H 3850 3900 50  0001 C CNN
-F 3 "" H 3850 3900 50  0001 C CNN
-	1    3850 3900
+P 3850 3800
+F 0 "#PWR053" H 3850 3550 50  0001 C CNN
+F 1 "GND" H 3855 3627 50  0000 C CNN
+F 2 "" H 3850 3800 50  0001 C CNN
+F 3 "" H 3850 3800 50  0001 C CNN
+	1    3850 3800
 	1    0    0    -1
 $EndComp
@@
 L power:+3.3V #PWR048
 U 1 1 5CEB4D06
-P 3300 2900
-F 0 "#PWR048" H 3300 2750 50  0001 C CNN
-F 1 "+3.3V" H 3150 3050 50  0000 C CNN
-F 2 "" H 3300 2900 50  0001 C CNN
-F 3 "" H 3300 2900 50  0001 C CNN
-	1    3300 2900
-	1    0    0    -1
-$EndComp
-Wire Wire Line
-	3300 2900 3300 3200
-Wire Wire Line
-	3300 3200 3950 3200
+P 3700 2750
+F 0 "#PWR048" H 3700 2600 50  0001 C CNN
+F 1 "+3.3V" H 3750 2900 50  0000 C CNN
+F 2 "" H 3700 2750 50  0001 C CNN
+F 3 "" H 3700 2750 50  0001 C CNN
+	1    3700 2750
+	1    0    0    -1
+$EndComp
+Wire Wire Line
+	3700 2750 3700 2850
+Wire Wire Line
+	3700 2850 3950 2850
 $Comp
 L Device:R R17
@@
 	-1   0    0    1
 $EndComp
-Text Label 3400 3300 0    50   ~ 0
+Text Label 3600 2950 0    50   ~ 0
 PROG_RTS
-Text Label 3400 3400 0    50   ~ 0
+Text Label 3600 3050 0    50   ~ 0
 PROG_DTR
-Text Label 3400 3500 0    50   ~ 0
+Text Label 3600 3150 0    50   ~ 0
 PROG_RXD
-Text Label 3400 3600 0    50   ~ 0
+Text Label 3600 3250 0    50   ~ 0
 PROG_TXD
 Wire Wire Line
@@
 L Connector_Generic:Conn_01x08 J1
 U 1 1 5EA4F7A2
-P 4150 3300
-F 0 "J1" H 4100 3850 50  0000 L CNN
-F 1 "Conn_01x08" H 3950 3750 50  0000 L CNN
-F 2 "Connector_PinSocket_2.54mm:PinSocket_1x08_P2.54mm_Vertical" H 4150 3300 50  0001 C CNN
-F 3 "~" H 4150 3300 50  0001 C CNN
-	1    4150 3300
+P 4150 3150
+F 0 "J1" H 4100 3700 50  0000 L CNN
+F 1 "Conn_01x08" H 3950 3600 50  0000 L CNN
+F 2 "Connector_PinSocket_2.54mm:PinSocket_1x08_P2.54mm_Vertical" H 4150 3150 50  0001 C CNN
+F 3 "~" H 4150 3150 50  0001 C CNN
+	1    4150 3150
 	1    0    0    -1
 $EndComp
@@
 L power:VBUS #PWR0105
 U 1 1 5EA736C0
-P 3500 2900
-F 0 "#PWR0105" H 3500 2750 50  0001 C CNN
-F 1 "VBUS" H 3550 3050 50  0000 C CNN
-F 2 "" H 3500 2900 50  0001 C CNN
-F 3 "" H 3500 2900 50  0001 C CNN
-	1    3500 2900
+P 3500 2750
+F 0 "#PWR0105" H 3500 2600 50  0001 C CNN
+F 1 "VBUS" H 3400 2900 50  0000 C CNN
+F 2 "" H 3500 2750 50  0001 C CNN
+F 3 "" H 3500 2750 50  0001 C CNN
+	1    3500 2750
 	1    0    0    -1
 $EndComp
@@
 	2450 5100 3350 5100
 Wire Wire Line
-	3150 4800 3150 3400
-Wire Wire Line
-	3150 3400 3950 3400
+	3150 4800 3150 3050
+Wire Wire Line
+	3150 3050 3950 3050
 Wire Wire Line
 	2850 4800 3150 4800
@@
 Connection ~ 1200 4800
 Wire Wire Line
-	3250 4900 3250 3500
+	3250 4900 3250 3150
 Wire Wire Line
 	2450 4900 3250 4900
 Wire Wire Line
-	3250 3500 3950 3500
-Wire Wire Line
-	3350 5100 3350 3600
-Wire Wire Line
-	3350 3600 3950 3600
+	3250 3150 3950 3150
+Wire Wire Line
+	3350 5100 3350 3250
+Wire Wire Line
+	3350 3250 3950 3250
 Wire Notes Line
-	3900 3150 3900 3750
+	3900 2800 3900 3400
 Wire Notes Line
-	3900 3750 4250 3750
+	3900 3400 4250 3400
 Wire Notes Line
-	4250 3750 4250 3150
+	4250 3400 4250 2800
 Wire Notes Line
-	4250 3150 3900 3150
+	4250 2800 3900 2800
 Wire Wire Line
 	5300 7650 5300 7200
@@
 	10100 2050 10100 1600
 $Comp
-L VCOMLCD-rescue:74LVC4245A-Logic_LevelTranslator U3
+L VCOMLCD-rescue:74LVC4245A-Logic_LevelTranslator-VCOMLCD-rescue U3
 U 1 1 5D78A3BC
 P 6950 5050
@@
 	2450 5300 5050 5300
 Wire Wire Line
-	2950 3300 2950 3700
+	2950 2950 2950 3700
 Wire Wire Line
 	2950 3700 1200 3700
 Wire Wire Line
-	2950 3300 3950 3300
+	2950 2950 3950 2950
 Wire Wire Line
 	1150 2850 1150 3150
@@
 NoConn ~ 1100 1700
 Wire Wire Line
-	3500 2900 3500 3000
-Wire Wire Line
-	3500 3000 3950 3000
-Wire Wire Line
-	3850 3700 3850 3900
-Wire Wire Line
-	3850 3700 3850 3100
-Wire Wire Line
-	3850 3100 3950 3100
-Connection ~ 3850 3700
+	3850 3350 3850 3450
+Wire Wire Line
+	3850 3450 3950 3450
 $Comp
 L Device:LED D1
@@
 	-1   0    0    -1
 $EndComp
+Connection ~ 3850 3450
+Wire Wire Line
+	3850 3450 3850 3800
+Wire Wire Line
+	3500 3550 3950 3550
+Wire Wire Line
+	3500 2750 3500 3550
 $EndSCHEMATC
