File: VCOMLCD.sch (KiCad schematic (older format))
At the start: 49 parts, among them J1 Screw_Terminal_01x02, J2 USB_B_Mini, J3 Conn_01x05, J4 Conn_01x03, J5 Conn_01x06, Q1 BC847, SW1 SYS_RST, SW2 BTN, U1 MCP73831-2-OT, U2 MCP1700-3302E_SOT23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

Commit message: final rev1 files
Parts:
- R12: value R -> 10k
Other:
- note added: "Rev. 1\n-Initial release\nRev.2\n- Selected proper LCD footprint\n- added dedicated 5V pin\n- removed R1/R2 solderbridges\n- addded pwr/status LEDs\n"
Changed lines of the file:
@@
 P 10800 3750
 F 0 "R12" H 10730 3704 50  0000 R CNN
-F 1 "R" H 10730 3795 50  0000 R CNN
+F 1 "10k" H 10730 3795 50  0000 R CNN
 F 2 "Resistor_SMD:R_0603_1608Metric_Pad1.05x0.95mm_HandSolder" V 10730 3750 50  0001 C CNN
 F 3 "~" H 10800 3750 50  0001 C CNN
@@
 Wire Wire Line
 	7400 1950 7400 2450
+Text Notes 9150 1150 0    50   ~ 0
+Rev. 1\n-Initial release\nRev.2\n- Selected proper LCD footprint\n- added dedicated 5V pin\n- removed R1/R2 solderbridges\n- addded pwr/status LEDs\n
 $EndSCHEMATC
